File: Acid_Drip_PCB- Kicad/Acid_Synth/Acid_Synth.kicad_pcb (KiCad board)
At the start: 2 copper layers, 169 x 114.4 mm, 43 parts, among them J1 Sync_In, J2 Output, J3 Conn_01x02_Socket, SW17 SW_SPDT, SW18 SW_SPDT, U1 TFT_2.8in_ILI9341

Commit message: Cleanup of PCB
Parts:
- SW17: value SW_SPDT -> POWER
- moved C9 12.0 mm to (63.0, 83.2)
- moved C6 2.03 mm to (150.3, 47.4), turned to 0 degrees
Routing:
- net OUTPUT: track 162.6 -> 99.6 mm, vias 0 -> 1
- net GND: track 1.02 -> 52.7 mm, vias 0 -> 214
- net SW3: track 51.5 -> 101.3 mm, vias 0 -> 1
- net SW13: track 221.9 -> 181.4 mm
- net SW14: track 228.9 -> 188.6 mm, vias 0 -> 1
- net Decay: track 159.2 -> 120.1 mm
- net SW8: track 263.3 -> 224.6 mm, vias 0 -> 2
- net SW7: track 240.3 -> 201.7 mm, vias 0 -> 2
- net W16: track 208.7 -> 246.9 mm, vias 0 -> 2
- net SW12: track 203.8 -> 167.1 mm
- net SW2: track 44.5 -> 79.6 mm, vias 0 -> 1
- net SW6: track 215.0 -> 181.5 mm, vias 0 -> 2
- net SW11: track 184.0 -> 152.5 mm
- net SW10: track 173.3 -> 143.1 mm, vias 0 -> 2
- net SW5: track 184.8 -> 154.9 mm, vias 0 -> 2
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
Commit message: ready for test
Parts:
- moved SW3 21.4 mm to (119.9, 106.8)
- moved SW5 21.4 mm to (158.5, 106.8)
- moved SW6 21.4 mm to (177.8, 106.8)
- moved SW7 21.4 mm to (197.1, 106.8)
- moved SW8 21.4 mm to (216.4, 106.8)
- moved C5 21.4 mm to (163.1, 59.0)
- moved C6 21.4 mm to (168.3, 59.0)
- moved C7 21.4 mm to (163.5, 67.7)
- moved J1 21.4 mm to (165.8, 41.4)
- moved J2 21.4 mm to (203.9, 41.4)
- moved SW17 21.4 mm to (218.1, 47.9)
- moved SW18 21.4 mm to (151.7, 47.9)
- moved level1 21.4 mm to (182.4, 55.4)
- moved C1 21.4 mm to (159.8, 67.9)
- moved C2 21.4 mm to (159.8, 64.6)
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Routing:
- net +3.3V: track 247.3 -> 243.6 mm, vias 0 -> 1
- net SW8: track 224.6 -> 222.4 mm
- net SW7: track 201.7 -> 200.2 mm
- net GND: vias 214 -> 256
Other:
- board text added: "10nf"
