File: Acid_Drip_PCB- Kicad/Acid_Synth/Acid_Synth.kicad_sch (KiCad schematic)
At the start: 37 parts, among them J1 Sync_In, J2 Output, J3 Conn_01x02_Socket, SW17 SW_SPDT, SW18 SW_SPDT, U1 TFT_2.8in_ILI9341

Commit message: ready for test
Parts:
- SW1, SW10, SW11, SW12, SW13, SW14, SW15, SW16, SW2, SW3, SW4, SW5, SW6, SW7, SW8, SW9: value ~ -> (none)
